File: variants/business-card-v1/hardware/Insert-Coin-Business-Card.kicad_pcb (KiCad board)
At the start: 2 copper layers, 88.9 x 50.8 mm, 52 parts, among them J1 Conn_01x02, Q1 CJ3400, Q10 CJ3400, Q2 CJ3400, Q3 CJ3400, Q4 CJ3400, Q5 CJ3400, Q7 CJ3400, Q8 CJ3400, Q9 CJ3400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

Commit message: PCB File Updated
- updated the pcb layout and mic choice to have it be economy parts for jlc.
- removed the VCC testpoint
- change UPDI & GND testpoint to be ducky shape
Parts:
- removed MIC1: ZTS6156, KiCadPartFinder:MIC-SMD_3P-L2.8-W1.9_ZTS6056
- removed R1, R2, R3, R4, R5, R6: 10kΩ, PCM_Resistor_SMD_AKL:R_Array_Convex_4x0402
- removed TP2: 1.0mm, PCM_SparkFun-Connector:TestPoint-1.0mm
- removed kibuzzard-6A02E010: G***, kibuzzard-6A02E010
- added U3: LMA2718B381-OA7, KiCadPartFinder:MIC-SMD_4P-L2.8-W1.9_LMA2718B381-OA7, B.Cu at (190.5, 75.3)
- TP1, TP3: footprint PCM_SparkFun-Connector:TestPoint-1.0mm -> DavidLib_Graphics:DUCKY_ICON_2.54_Spacing
- moved kibuzzard-6A02DFFE 0.26 mm to (133.8, 80.3)
- moved kibuzzard-6A02E019 0.26 mm to (131.2, 80.4)
- moved TP1 0.25 mm to (132.0, 82.7), turned to 180 degrees
- moved TP3 0.25 mm to (129.5, 82.7), turned to 180 degrees
Connections:
- LED1 pad 2: Net-(LED1-A) -> VCC
- LED10 pad 2: Net-(LED10-A) -> VCC
- LED11 pad 2: Net-(LED11-A) -> VCC
- LED12 pad 2: Net-(LED12-A) -> VCC
- LED13 pad 2: Net-(LED13-A) -> VCC
- LED14 pad 2: Net-(LED14-A) -> VCC
- LED15 pad 2: Net-(LED15-A) -> VCC
- LED16 pad 2: Net-(LED16-A) -> VCC
- LED17 pad 2: Net-(LED17-A) -> VCC
- LED18 pad 2: Net-(LED18-A) -> VCC
- LED19 pad 2: Net-(LED19-A) -> VCC
- LED2 pad 2: Net-(LED2-A) -> VCC
- LED20 pad 2: Net-(LED20-A) -> VCC
- LED21 pad 2: Net-(LED21-A) -> VCC
- LED22 pad 2: Net-(LED22-A) -> VCC
- LED23 pad 2: Net-(LED23-A) -> VCC
- LED24 pad 2: Net-(LED24-A) -> VCC
- LED3 pad 2: Net-(LED3-A) -> VCC
- LED4 pad 2: Net-(LED4-A) -> VCC
- LED5 pad 2: Net-(LED5-A) -> VCC
- LED6 pad 2: Net-(LED6-A) -> VCC
- LED7 pad 2: Net-(LED7-A) -> VCC
- LED8 pad 2: Net-(LED8-A) -> VCC
- LED9 pad 2: Net-(LED9-A) -> VCC
Routing:
- net VCC: track 195.5 -> 503.1 mm, vias 0 -> 8
- net Net-(LED24-A): track 31.5 -> 0.00 mm
- net Net-(LED8-A): track 24.3 -> 0.00 mm
- net Net-(LED4-A): track 21.5 -> 0.00 mm
- net Net-(LED23-A): track 19.9 -> 0.00 mm
- net Net-(LED16-A): track 19.4 -> 0.00 mm, vias 2 -> 0
- net Net-(LED20-A): track 19.2 -> 0.00 mm, vias 2 -> 0
- net Net-(LED6-A): track 18.1 -> 0.00 mm
- net Net-(LED11-A): track 17.8 -> 0.00 mm
- net Net-(LED19-A): track 17.3 -> 0.00 mm, vias 2 -> 0
- net Net-(LED2-A): track 17.2 -> 0.00 mm
- net Net-(LED15-A): track 16.4 -> 0.00 mm, vias 2 -> 0
- net Net-(LED12-A): track 16.4 -> 0.00 mm
- net Net-(LED10-A): track 8.52 -> 0.00 mm
- net Net-(LED22-A): track 8.35 -> 0.00 mm
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