File: variants/business-card-v1/hardware/Ducky Business Card V0-1/Insert-Coin-Business-Card.kicad_pcb (KiCad board)
At the start: 2 copper layers, 88.9 x 50.8 mm, 44 parts, among them J1 Conn_01x02, Q1 CJ3400, Q10 CJ3400, Q2 CJ3400, Q3 CJ3400, Q4 CJ3400, Q5 CJ3400, Q7 CJ3400, Q8 CJ3400, Q9 CJ3400, U1 ATtiny1616-M, U2 ST25DV04K-IER8C3, U3 LMA2718B381-OA7

Commit message: WIP: hardware V0-1 to V0-3 folders, production-nfc config tweak
Parts:
- moved kibuzzard-6A02E019 5.55 mm to (136.7, 80.3)
- moved TP3 5.18 mm to (134.7, 82.6)
- moved kibuzzard-6A02DFFE 0.50 mm to (134.3, 80.1)
- moved LED22 0.28 mm to (188.7, 62.4)
- moved LED21 0.28 mm to (180.1, 62.3)
- moved LED24 0.18 mm to (180.0, 70.7)
- moved TP1 0.14 mm to (132.1, 82.6)
