File: variants/business-card-v1/hardware/Ducky-Business-Card-V0-2/Ducky-Business-Card-V0-2.kicad_sch (KiCad schematic)
At the start: 42 parts, among them J1 Conn_01x02, Q1 CJ3400, Q10 CJ3400, Q2 CJ3400, Q3 CJ3400, Q4 CJ3400, Q5 CJ3400, Q7 CJ3400, Q8 CJ3400, Q9 CJ3400, U1 ATtiny1616-M, U2 ST25DV04K-IER8C3, U3 LMA2718B381-OA7

Commit message: WIP: hardware V0-1 to V0-3 folders, production-nfc config tweak
Parts:
- LED21, LED22: LCSC C965861 -> C965860
- LED23, LED24: Attrition Qty C965860 -> (none); LCSC C965860 -> C965861
Other:
- company: (none) -> ByProduct Lab
- title: (none) -> Ducky Business Card
